File: ESP32-Based-Power-Monitoring-System/ESP32_Based_Power_Monitoring_System/ESP32_Based_Power_Monitoring_System.kicad_pcb (KiCad board)
At the start: 4 copper layers, 133.3 x 58.2 mm, 161 parts, among them J1 12V/5A, J10 Barrel_Jack_Switch, J11 Barrel_Jack_Switch, J2 USB_C, J3 OLED DISPLAY, J4 Barrel_Jack_Switch, J5 Barrel_Jack_Switch, J6 Barrel_Jack_Switch, J7 Barrel_Jack_Switch, J8 Barrel_Jack_Switch, J9 Barrel_Jack_Switch, Q1 BC817, Q10 QM6015D, Q11 QM6006D, Q12 QM6006D, Q13 QM6006D, Q14 QM6006D, Q15 QM6015D, Q16 QM6015D, Q17 QM6015D, Q18 QM6015D, Q2 BC817, Q3 QM6006D, Q4 QM6006D, Q5 QM6006D, Q6 QM6006D, Q7 QM6015D, Q8 QM6015D, Q9 QM6015D, SW1 RotaryEncoder_Switch_MP, SW2 SW_Push, SW3 SW_Push, U10 INA219AxD, U11 INA219AxD, U12 INA219AxD, U13 INA219AxD, U14 tps54331, U2 LM1084-3.3, U3 LM1084-ADJ, U4 CP2102N-Axx-xQFN28, U5 ESP32-WROOM-32UE, U6 INA219AxD, U7 INA219AxD, U8 INA219AxD, U9 INA219AxD

Commit message: Second Commit
Parts:
- D5: footprint Diode_SMD:D_SMA -> Diode_SMD:D_SMF
- moved R23 3.17 mm to (78.0, 105.2), turned to 0 degrees
- moved R25 2.68 mm to (77.5, 98.8)
- moved L1 1.34 mm to (46.8, 83.0)
- moved D5 1.04 mm to (47.1, 87.1)
Routing:
- net /IIC_SCK: track 0.00 -> 225.1 mm, vias 0 -> 16
- net /IIC_SDA: track 2.54 -> 223.8 mm, vias 0 -> 15
- net /ENC_S2: track 3.29 -> 77.9 mm, vias 0 -> 2
- net /ESP_EN8: track 1.83 -> 73.9 mm, vias 0 -> 2
- net /ESP_EN3: track 1.62 -> 73.5 mm, vias 0 -> 4
- net /ESP_EN4: track 1.80 -> 59.4 mm, vias 0 -> 2
- net /ESP_EN6: track 2.02 -> 59.3 mm, vias 0 -> 2
- net /ESP_EN5: track 1.79 -> 58.2 mm, vias 0 -> 2
- net /ENC_B: track 4.59 -> 59.8 mm, vias 0 -> 2
- net /ENC_A: track 4.69 -> 59.8 mm, vias 0 -> 2
- net GND: track 265.5 -> 314.4 mm, vias 70 -> 93
- net /ESP_EN7: track 1.61 -> 49.5 mm, vias 0 -> 2
- net /ESP_EN: track 8.02 -> 42.5 mm, vias 0 -> 2
- net /ESP_EN2: track 1.62 -> 34.0 mm, vias 0 -> 2
- net /ESP_EN1: track 1.68 -> 33.7 mm, vias 0 -> 2
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